Commit message: fix: 第 1-10 轮迭代修复
Round 1: Gazebo 颜色参数化 (chassis.xacro 添加 gazebo_r/g/b 参数)
Round 2: 消除 pi 重复传递 (mecanum_wheel 内部定义)
Round 3: 所有传感器/机械臂添加碰撞体
Round 4: robot_state.py 文档字符串更新
Round 5: 删除 swarm.launch.py 死参数 use_sim
Round 6-8: 代码审查无新问题
Round 9: 修复三个 Makefile 死路径 (../../shared/protocol)
Round 10: 全量测试通过 (9/9)

File: swarm_bringup/urdf/carrier/carrier.urdf.xacro (robot description, xacro)
@@ -14,18 +14,18 @@
     wheel_radius="0.065" wheel_pos_z="-0.048"
     mesh_file="package://swarm_bringup/meshes/shared/chassis.dae"
-    body_material="body_green"/>
+    body_material="body_green" gazebo_r="0.15" gazebo_g="0.75" gazebo_b="0.30"/>
   <!-- 麦轮 -->
   <xacro:mecanum_wheel side="front_left"  radius="0.065" width="0.035"
     pos_x="0.185" pos_y="0.170" pos_z="-0.048" mass="0.25"
-    mesh_file="package://swarm_bringup/meshes/shared/tire.dae" pi="${pi}"/>
+    mesh_file="package://swarm_bringup/meshes/shared/tire.dae"/>
   <xacro:mecanum_wheel side="front_right" radius="0.065" width="0.035"
     pos_x="0.185" pos_y="-0.170" pos_z="-0.048" mass="0.25"
-    mesh_file="package://swarm_bringup/meshes/shared/tire.dae" pi="${pi}"/>
+    mesh_file="package://swarm_bringup/meshes/shared/tire.dae"/>
   <xacro:mecanum_wheel side="rear_left"   radius="0.065" width="0.035"
     pos_x="-0.185" pos_y="0.170" pos_z="-0.048" mass="0.25"
-    mesh_file="package://swarm_bringup/meshes/shared/tire.dae" pi="${pi}"/>
+    mesh_file="package://swarm_bringup/meshes/shared/tire.dae"/>
   <xacro:mecanum_wheel side="rear_right"  radius="0.065" width="0.035"
     pos_x="-0.185" pos_y="-0.170" pos_z="-0.048" mass="0.25"
-    mesh_file="package://swarm_bringup/meshes/shared/tire.dae" pi="${pi}"/>
+    mesh_file="package://swarm_bringup/meshes/shared/tire.dae"/>
   <!-- Carrier 专属 -->
   <xacro:supply_bay/>

File: swarm_bringup/urdf/common/chassis.xacro (robot description, xacro)
@@ -6,5 +6,5 @@
 -->
 <robot xmlns:xacro="http://ros.org/wiki/xacro" xmlns:gz="http://gazebosim.org/schema">
-  <xacro:macro name="chassis" params="length width height mass wheel_radius wheel_pos_z mesh_file body_material">
+  <xacro:macro name="chassis" params="length width height mass wheel_radius wheel_pos_z mesh_file body_material gazebo_r gazebo_g gazebo_b">
     <!-- base_footprint (地面参考点) -->
     <link name="base_footprint"/>
@@ -40,10 +40,10 @@
       </inertial>
     </link>
-    <!-- Gazebo 材质 -->
+    <!-- Gazebo 材质 (参数化颜色) -->
     <gazebo reference="base_link">
       <visual>
         <material>
-          <ambient>0.18 0.42 0.82 1.0</ambient>
-          <diffuse>0.18 0.42 0.82 1.0</diffuse>
+          <ambient>${gazebo_r} ${gazebo_g} ${gazebo_b} 1.0</ambient>
+          <diffuse>${gazebo_r} ${gazebo_g} ${gazebo_b} 1.0</diffuse>
           <specular>0.3 0.3 0.3 1.0</specular>
           <emissive>0.0 0.0 0.0 0.0</emissive>

File: swarm_bringup/urdf/common/mecanum_wheel.xacro (robot description, xacro)
@@ -6,5 +6,6 @@
 -->
 <robot xmlns:xacro="http://ros.org/wiki/xacro" xmlns:gz="http://gazebosim.org/schema">
-  <xacro:macro name="mecanum_wheel" params="side radius width pos_x pos_y pos_z mass mesh_file pi">
+  <xacro:macro name="mecanum_wheel" params="side radius width pos_x pos_y pos_z mass mesh_file">
+    <xacro:property name="pi" value="3.14159265358979"/>
     <link name="${side}_wheel_link">
       <visual>

File: swarm_bringup/urdf/common/sensors.xacro (robot description, xacro)
@@ -20,4 +20,5 @@
     <link name="livox_link">
       <visual><geometry><box size="0.065 0.065 0.052"/></geometry><material name="dark"/></visual>
+      <collision><geometry><box size="0.065 0.065 0.052"/></geometry></collision>
     </link>
     <joint name="livox_joint" type="fixed">
@@ -30,4 +31,5 @@
     <link name="realsense_link">
       <visual><geometry><box size="0.124 0.026 0.029"/></geometry><material name="dark"/></visual>
+      <collision><geometry><box size="0.124 0.026 0.029"/></geometry></collision>
     </link>
     <joint name="realsense_joint" type="fixed">
@@ -40,4 +42,5 @@
     <link name="radar_link">
       <visual><geometry><box size="0.065 0.045 0.012"/></geometry><material name="dark"/></visual>
+      <collision><geometry><box size="0.065 0.045 0.012"/></geometry></collision>
     </link>
     <joint name="radar_joint" type="fixed">
@@ -68,4 +71,5 @@
     <link name="thermal_link">
       <visual><geometry><box size="0.035 0.035 0.025"/></geometry><material name="dark"/></visual>
+      <collision><geometry><box size="0.035 0.035 0.025"/></geometry></collision>
     </link>
     <joint name="thermal_joint" type="fixed">
@@ -78,4 +82,5 @@
     <link name="arm_base">
       <visual><geometry><cylinder radius="0.035" length="0.015"/></geometry><material name="dark"/></visual>
+      <collision><geometry><cylinder radius="0.035" length="0.015"/></geometry></collision>
     </link>
     <joint name="arm_base_j" type="fixed">
@@ -85,4 +90,5 @@
     <link name="arm_link1">
       <visual><geometry><box size="0.035 0.035 0.15"/></geometry><material name="arm_color"/></visual>
+      <collision><geometry><box size="0.035 0.035 0.15"/></geometry></collision>
       <inertial><origin xyz="0 0 0.075"/><mass value="0.5"/><inertia ixx="0.001" ixy="0" ixz="0" iyy="0.001" iyz="0" izz="0.0002"/></inertial>
     </link>
@@ -94,4 +100,5 @@
     <link name="arm_link2">
       <visual><geometry><box size="0.028 0.028 0.12"/></geometry><material name="arm_color"/></visual>
+      <collision><geometry><box size="0.028 0.028 0.12"/></geometry></collision>
       <inertial><origin xyz="0 0 0.06"/><mass value="0.35"/><inertia ixx="0.0005" ixy="0" ixz="0" iyy="0.0005" iyz="0" izz="0.0001"/></inertial>
     </link>
@@ -103,4 +110,5 @@
     <link name="gripper_base">
       <visual><geometry><box size="0.035 0.030 0.015"/></geometry><material name="dark"/></visual>
+      <collision><geometry><box size="0.035 0.030 0.015"/></geometry></collision>
     </link>
     <joint name="gripper_j" type="revolute">
@@ -126,4 +134,5 @@
     <link name="router_box">
       <visual><geometry><box size="0.10 0.08 0.025"/></geometry><material name="dark"/></visual>
+      <collision><geometry><box size="0.10 0.08 0.025"/></geometry></collision>
     </link>
     <joint name="router_box_j" type="fixed">

File: swarm_bringup/urdf/scout/scout.urdf.xacro (robot description, xacro)
@@ -15,18 +15,18 @@
     wheel_radius="0.048" wheel_pos_z="-0.040"
     mesh_file="package://swarm_bringup/meshes/shared/chassis.dae"
-    body_material="body_blue"/>
+    body_material="body_blue" gazebo_r="0.18" gazebo_g="0.42" gazebo_b="0.82"/>
   <!-- 麦轮 (4个) -->
   <xacro:mecanum_wheel side="front_left"  radius="0.048" width="0.028"
     pos_x="0.160" pos_y="0.140" pos_z="-0.040" mass="0.15"
-    mesh_file="package://swarm_bringup/meshes/shared/tire.dae" pi="${pi}"/>
+    mesh_file="package://swarm_bringup/meshes/shared/tire.dae"/>
   <xacro:mecanum_wheel side="front_right" radius="0.048" width="0.028"
     pos_x="0.160" pos_y="-0.140" pos_z="-0.040" mass="0.15"
-    mesh_file="package://swarm_bringup/meshes/shared/tire.dae" pi="${pi}"/>
+    mesh_file="package://swarm_bringup/meshes/shared/tire.dae"/>
   <xacro:mecanum_wheel side="rear_left"   radius="0.048" width="0.028"
     pos_x="-0.160" pos_y="0.140" pos_z="-0.040" mass="0.15"
-    mesh_file="package://swarm_bringup/meshes/shared/tire.dae" pi="${pi}"/>
+    mesh_file="package://swarm_bringup/meshes/shared/tire.dae"/>
   <xacro:mecanum_wheel side="rear_right"  radius="0.048" width="0.028"
     pos_x="-0.160" pos_y="-0.140" pos_z="-0.040" mass="0.15"
-    mesh_file="package://swarm_bringup/meshes/shared/tire.dae" pi="${pi}"/>
+    mesh_file="package://swarm_bringup/meshes/shared/tire.dae"/>
   <!-- Scout 传感器 -->
   <xacro:lidar_2d x="0.06" y="0" z="0.20"/>

File: swarm_bringup/urdf/specialist/specialist.urdf.xacro (robot description, xacro)
@@ -14,18 +14,18 @@
     wheel_radius="0.055" wheel_pos_z="-0.044"
     mesh_file="package://swarm_bringup/meshes/shared/chassis.dae"
-    body_material="body_orange"/>
+    body_material="body_orange" gazebo_r="0.92" gazebo_g="0.52" gazebo_b="0.12"/>
   <!-- 麦轮 -->
   <xacro:mecanum_wheel side="front_left"  radius="0.055" width="0.030"
     pos_x="0.150" pos_y="0.150" pos_z="-0.044" mass="0.20"
-    mesh_file="package://swarm_bringup/meshes/shared/tire.dae" pi="${pi}"/>
+    mesh_file="package://swarm_bringup/meshes/shared/tire.dae"/>
   <xacro:mecanum_wheel side="front_right" radius="0.055" width="0.030"
     pos_x="0.150" pos_y="-0.150" pos_z="-0.044" mass="0.20"
-    mesh_file="package://swarm_bringup/meshes/shared/tire.dae" pi="${pi}"/>
+    mesh_file="package://swarm_bringup/meshes/shared/tire.dae"/>
   <xacro:mecanum_wheel side="rear_left"   radius="0.055" width="0.030"
     pos_x="-0.150" pos_y="0.150" pos_z="-0.044" mass="0.20"
-    mesh_file="package://swarm_bringup/meshes/shared/tire.dae" pi="${pi}"/>
+    mesh_file="package://swarm_bringup/meshes/shared/tire.dae"/>
   <xacro:mecanum_wheel side="rear_right"  radius="0.055" width="0.030"
     pos_x="-0.150" pos_y="-0.150" pos_z="-0.044" mass="0.20"
-    mesh_file="package://swarm_bringup/meshes/shared/tire.dae" pi="${pi}"/>
+    mesh_file="package://swarm_bringup/meshes/shared/tire.dae"/>
   <!-- Specialist 专属 -->
   <xacro:thermal_camera x="0.20" y="-0.05" z="0.08"/>
