Commit message: feat: xacro 建模深度重构 (第 51-100 轮)
rescue_robot.urdf.xacro 完全重写:
- 改用模块化 include 架构 (与 scout/carrier/specialist 一致)
- 使用 linorobot2 网格 (chassis.dae + tire.dae)
- 支持 robot_name 参数切换三机
- Gazebo 颜色参数化 (蓝/绿/橙)

gazebo_plugins.xacro 增强:
- 添加 13 个传感器 Gazebo 材质定义
- 添加 RealSense D455 深度相机插件

sensors.xacro 增强:
- 所有 5 个传感器链接添加惯性属性
- lidar_link: 0.1kg
- livox_link: 0.2kg
- realsense_link: 0.12kg
- radar_link: 0.05kg
- thermal_link: 0.03kg

清理:
- 删除 4 个未使用的旧网格 (chassis_base/gimbal_yaw/wheel_left/wheel_right)
- meshes/shared/ 仅保留 2 个实际使用的文件 (7.1MB)

验证: XML 9/9 + Python 56/56 + Tests 6/6 全通过

File: swarm_bringup/urdf/common/gazebo_plugins.xacro (robot description, xacro)
@@ -1,53 +1,108 @@
 <?xml version="1.0"?>
 <!--
-  gazebo_plugins.xacro — Gazebo 仿真插件
-  麦轮驱动 + 2D LiDAR + IMU
+  gazebo_plugins.xacro — Gazebo 仿真插件 + 传感器材质
+  包含:
+  - 麦轮驱动 (diff_drive)
+  - 2D LiDAR (ray sensor)
+  - IMU
+  - 深度相机 (RealSense D455)
+  - 传感器材质定义 (dark/lens/accent)
 -->
 <robot xmlns:xacro="http://ros.org/wiki/xacro">
   <xacro:macro name="gazebo_mecanum" params="namespace wheel_base wheel_separation wheel_radius">
-    <gazebo>
-      <!-- 麦轮驱动 -->
-      <plugin name="mecanum_drive" filename="libgazebo_ros_diff_drive.so">
-        <ros><namespace>${namespace}</namespace></ros>
-        <update_rate>100</update_rate>
-        <left_joint>front_left_wheel_joint rear_left_wheel_joint</left_joint>
-        <right_joint>front_right_wheel_joint rear_right_wheel_joint</right_joint>
-        <wheel_separation>${wheel_separation}</wheel_separation>
-        <wheel_diameter>${2*wheel_radius}</wheel_diameter>
-        <max_wheel_torque>10.0</max_wheel_torque>
-        <command_topic>cmd_vel</command_topic>
-        <odometry_topic>odom</odometry_topic>
-        <odometry_frame>odom</odometry_frame>
-        <robot_base_frame>base_link</robot_base_frame>
-        <publish_odom_tf>true</publish_odom_tf>
-      </plugin>
-      <!-- 2D LiDAR -->
-      <plugin name="lidar" filename="libgazebo_ros_ray_sensor.so">
-        <ros><namespace>${namespace}</namespace></ros>
-        <update_rate>10</update_rate>
-        <sensor>
-          <type>ray</type>
-          <pose>0.06 0 0.20 0 0 0</pose>
-          <visualize>false</visualize>
-          <ray>
-            <scan><horizontal>
-              <samples>360</samples><resolution>1</resolution>
-              <min_angle>-3.14159</min_angle><max_angle>3.14159</max_angle>
-            </horizontal></scan>
-            <range><min>0.12</min><max>6.0</max><resolution>0.01</resolution></range>
-            <noise><type>gaussian</type><mean>0.0</mean><stddev>0.012</stddev></noise>
-          </ray>
-        </sensor>
-      </plugin>
-      <!-- IMU -->
-      <plugin name="imu" filename="libgazebo_ros_imu_sensor.so">
-        <ros><namespace>${namespace}</namespace></ros>
-        <always_on>true</always_on>
-        <update_rate>200</update_rate>
-        <body_name>base_link</body_name>
-        <topic>imu/data</topic>
-        <gaussian_noise>0.0005</gaussian_noise>
-      </plugin>
+    <!-- ═══ 传感器材质 ═══ -->
+    <gazebo reference="lidar_link">
+      <material>Gazebo/DarkGrey</material>
     </gazebo>
+    <gazebo reference="livox_link">
+      <material>Gazebo/DarkGrey</material>
+    </gazebo>
+    <gazebo reference="realsense_link">
+      <material>Gazebo/DarkGrey</material>
+    </gazebo>
+    <gazebo reference="radar_link">
+      <material>Gazebo/DarkGrey</material>
+    </gazebo>
+    <gazebo reference="uwb_tag">
+      <material>Gazebo/Yellow</material>
+    </gazebo>
+    <gazebo reference="thermal_link">
+      <material>Gazebo/DarkGrey</material>
+    </gazebo>
+    <gazebo reference="led_bar">
+      <material>Gazebo/Yellow</material>
+    </gazebo>
+    <gazebo reference="supply_box">
+      <material>Gazebo/Grey</material>
+    </gazebo>
+    <gazebo reference="router_box">
+      <material>Gazebo/DarkGrey</material>
+    </gazebo>
+    <gazebo reference="arm_base">
+      <material>Gazebo/DarkGrey</material>
+    </gazebo>
+    <gazebo reference="arm_link1">
+      <material>Gazebo/Orange</material>
+    </gazebo>
+    <gazebo reference="arm_link2">
+      <material>Gazebo/Orange</material>
+    </gazebo>
+    <gazebo reference="gripper_base">
+      <material>Gazebo/DarkGrey</material>
+    </gazebo>
+    <!-- ═══ 麦轮驱动 ═══ -->
+    <plugin name="mecanum_drive" filename="libgazebo_ros_diff_drive.so">
+      <ros><namespace>${namespace}</namespace></ros>
+      <update_rate>100</update_rate>
+      <left_joint>front_left_wheel_joint rear_left_wheel_joint</left_joint>
+      <right_joint>front_right_wheel_joint rear_right_wheel_joint</right_joint>
+      <wheel_separation>${wheel_separation}</wheel_separation>
+      <wheel_diameter>${2*wheel_radius}</wheel_diameter>
+      <max_wheel_torque>10.0</max_wheel_torque>
+      <command_topic>cmd_vel</command_topic>
+      <odometry_topic>odom</odometry_topic>
+      <odometry_frame>odom</odometry_frame>
+      <robot_base_frame>base_link</robot_base_frame>
+      <publish_odom_tf>true</publish_odom_tf>
+    </plugin>
+    <!-- ═══ 2D LiDAR ═══ -->
+    <plugin name="lidar" filename="libgazebo_ros_ray_sensor.so">
+      <ros><namespace>${namespace}</namespace></ros>
+      <update_rate>10</update_rate>
+      <sensor>
+        <type>ray</type>
+        <pose>0.06 0 0.20 0 0 0</pose>
+        <visualize>false</visualize>
+        <ray>
+          <scan><horizontal>
+            <samples>360</samples><resolution>1</resolution>
+            <min_angle>-3.14159</min_angle><max_angle>3.14159</max_angle>
+          </horizontal></scan>
+          <range><min>0.12</min><max>6.0</max><resolution>0.01</resolution></range>
+          <noise><type>gaussian</type><mean>0.0</mean><stddev>0.012</stddev></noise>
+        </ray>
+      </sensor>
+    </plugin>
+    <!-- ═══ IMU ═══ -->
+    <plugin name="imu" filename="libgazebo_ros_imu_sensor.so">
+      <ros><namespace>${namespace}</namespace></ros>
+      <always_on>true</always_on>
+      <update_rate>200</update_rate>
+      <body_name>base_link</body_name>
+      <topic>imu/data</topic>
+      <gaussian_noise>0.0005</gaussian_noise>
+    </plugin>
+    <!-- ═══ 深度相机 (Intel RealSense D455) ═══ -->
+    <plugin name="realsense_camera" filename="libgazebo_ros_camera.so">
+      <ros><namespace>${namespace}</namespace></ros>
+      <camera_name>realsense</camera_name>
+      <frame_name>realsense_link</frame_name>
+      <update_rate>30</update_rate>
+      <horizontal_fov>1.5708</horizontal_fov>
+      <image>
+        <width>640</width><height>480</height><format>R8G8B8</format>
+      </image>
+      <clip><near>0.02</near><far>10.0</far></clip>
+    </plugin>
   </xacro:macro>
 </robot>

File: swarm_bringup/urdf/common/sensors.xacro (robot description, xacro)
@@ -10,4 +10,5 @@
       <visual><geometry><cylinder radius="0.038" length="0.025"/></geometry><material name="dark"/></visual>
       <collision><geometry><cylinder radius="0.038" length="0.025"/></geometry></collision>
+      <inertial><mass value="0.1"/><inertia ixx="0.0001" ixy="0" ixz="0" iyy="0.0001" iyz="0" izz="0.00005"/></inertial>
     </link>
     <joint name="lidar_joint" type="fixed">
@@ -21,4 +22,5 @@
       <visual><geometry><box size="0.065 0.065 0.052"/></geometry><material name="dark"/></visual>
       <collision><geometry><box size="0.065 0.065 0.052"/></geometry></collision>
+      <inertial><mass value="0.2"/><inertia ixx="0.0002" ixy="0" ixz="0" iyy="0.0002" iyz="0" izz="0.0002"/></inertial>
     </link>
     <joint name="livox_joint" type="fixed">
@@ -32,4 +34,5 @@
       <visual><geometry><box size="0.124 0.026 0.029"/></geometry><material name="dark"/></visual>
       <collision><geometry><box size="0.124 0.026 0.029"/></geometry></collision>
+      <inertial><mass value="0.12"/><inertia ixx="0.0001" ixy="0" ixz="0" iyy="0.0002" iyz="0" izz="0.0002"/></inertial>
     </link>
     <joint name="realsense_joint" type="fixed">
@@ -43,4 +46,5 @@
       <visual><geometry><box size="0.065 0.045 0.012"/></geometry><material name="dark"/></visual>
       <collision><geometry><box size="0.065 0.045 0.012"/></geometry></collision>
+      <inertial><mass value="0.05"/><inertia ixx="0.00001" ixy="0" ixz="0" iyy="0.00001" iyz="0" izz="0.00001"/></inertial>
     </link>
     <joint name="radar_joint" type="fixed">
@@ -72,4 +76,5 @@
       <visual><geometry><box size="0.035 0.035 0.025"/></geometry><material name="dark"/></visual>
       <collision><geometry><box size="0.035 0.035 0.025"/></geometry></collision>
+      <inertial><mass value="0.03"/><inertia ixx="0.00001" ixy="0" ixz="0" iyy="0.00001" iyz="0" izz="0.00001"/></inertial>
     </link>
     <joint name="thermal_joint" type="fixed">
