Commit message: fix: 第 221-240 轮 — Nav2 参数 + 碰撞体补全
Nav2 参数修正 (三机统一):
- Carrier: max_vel_y 0→0.3, robot_radius 0.25→0.34
- Specialist: max_vel_y 0→0.3, robot_radius 0.25→0.29
- 三机麦轮横向运动全部启用

sensors.xacro 碰撞体+惯性补全:
- uwb_tag: 添加 collision + inertial
- led_bar: 添加 collision + inertial
- ant1/ant2: 添加 collision + inertial
- arm_base: 添加 inertial
- gripper_base: 添加 inertial
- router_box: 添加 inertial

全量测试: 7/7 通过

File: swarm_bringup/urdf/common/sensors.xacro (robot description, xacro)
@@ -65,4 +65,6 @@
     <link name="uwb_tag">
       <visual><geometry><box size="0.025 0.025 0.008"/></geometry><material name="accent"/></visual>
+      <collision><geometry><box size="0.025 0.025 0.008"/></geometry></collision>
+      <inertial><mass value="0.01"/><inertia ixx="0.000001" ixy="0" ixz="0" iyy="0.000001" iyz="0" izz="0.000001"/></inertial>
     </link>
     <joint name="uwb_tag_j" type="fixed">
@@ -88,4 +90,5 @@
       <visual><geometry><cylinder radius="0.035" length="0.015"/></geometry><material name="dark"/></visual>
       <collision><geometry><cylinder radius="0.035" length="0.015"/></geometry></collision>
+      <inertial><mass value="0.1"/><inertia ixx="0.00005" ixy="0" ixz="0" iyy="0.00005" iyz="0" izz="0.00003"/></inertial>
     </link>
     <joint name="arm_base_j" type="fixed">
@@ -116,4 +119,5 @@
       <visual><geometry><box size="0.035 0.030 0.015"/></geometry><material name="dark"/></visual>
       <collision><geometry><box size="0.035 0.030 0.015"/></geometry></collision>
+      <inertial><mass value="0.05"/><inertia ixx="0.00001" ixy="0" ixz="0" iyy="0.00001" iyz="0" izz="0.00001"/></inertial>
     </link>
     <joint name="gripper_j" type="revolute">
@@ -140,4 +144,5 @@
       <visual><geometry><box size="0.10 0.08 0.025"/></geometry><material name="dark"/></visual>
       <collision><geometry><box size="0.10 0.08 0.025"/></geometry></collision>
+      <inertial><mass value="0.15"/><inertia ixx="0.0001" ixy="0" ixz="0" iyy="0.0001" iyz="0" izz="0.00005"/></inertial>
     </link>
     <joint name="router_box_j" type="fixed">
@@ -145,7 +150,7 @@
       <origin xyz="0.12 0 0.08" rpy="0 0 0"/>
     </joint>
-    <link name="ant1"><visual><geometry><cylinder radius="0.005" length="0.12"/></geometry><material name="hub"/></visual></link>
+    <link name="ant1"><visual><geometry><cylinder radius="0.005" length="0.12"/></geometry><material name="hub"/></visual><collision><geometry><cylinder radius="0.005" length="0.12"/></geometry></collision><inertial><mass value="0.02"/><inertia ixx="0.000001" ixy="0" ixz="0" iyy="0.000001" iyz="0" izz="0.000001"/></inertial></link>
     <joint name="ant1_j" type="fixed"><parent link="router_box"/><child link="ant1"/><origin xyz="0.035 0.025 0.075" rpy="0 0 0"/></joint>
-    <link name="ant2"><visual><geometry><cylinder radius="0.005" length="0.12"/></geometry><material name="hub"/></visual></link>
+    <link name="ant2"><visual><geometry><cylinder radius="0.005" length="0.12"/></geometry><material name="hub"/></visual><collision><geometry><cylinder radius="0.005" length="0.12"/></geometry></collision><inertial><mass value="0.02"/><inertia ixx="0.000001" ixy="0" ixz="0" iyy="0.000001" iyz="0" izz="0.000001"/></inertial></link>
     <joint name="ant2_j" type="fixed"><parent link="router_box"/><child link="ant2"/><origin xyz="0.035 -0.025 0.075" rpy="0 0 0"/></joint>
   </xacro:macro>
@@ -154,4 +159,6 @@
     <link name="led_bar">
       <visual><geometry><box size="0.010 0.065 0.008"/></geometry><material name="accent"/></visual>
+      <collision><geometry><box size="0.010 0.065 0.008"/></geometry></collision>
+      <inertial><mass value="0.02"/><inertia ixx="0.000001" ixy="0" ixz="0" iyy="0.000001" iyz="0" izz="0.000001"/></inertial>
     </link>
     <joint name="led_bar_j" type="fixed">
